Commit message: added orbbec ros2 sdk

File: src/OrbbecSDK_ROS2/orbbec_description/urdf/gemini335Le.urdf.xacro (robot description, xacro)
@@ -24,5 +24,5 @@
     <visual>
       <origin
-        xyz="0 0 0"
+        xyz="-0.034005 -0.0475 -0.014048"
         rpy="0 0 0" />
       <geometry>
@@ -86,19 +86,6 @@
     </collision>
   </link>
-  <joint
-    name="base_Joint"
-    type="fixed">
-    <origin
-      xyz="0 0 0"
-      rpy="0 0 0" />
-    <parent
-      link="camera_botton_screw_frame" />
-    <child
-      link="camera_link" />
-    <axis
-      xyz="0 0 0" />
-  </joint>
-  <link
-    name="canera_right_IR_ROS_frame">
+    <link
+    name="camera_depth_frame">
     <inertial>
       <origin
@@ -115,43 +102,33 @@
         izz="4.8408E-09" />
     </inertial>
-    <visual>
-      <origin
-        xyz="0 0 0"
-        rpy="0 0 0" />
-      <geometry>
-        <mesh
-          filename="${mesh_path}canera_right_IR_ROS_frame.STL" />
-      </geometry>
-      <material
-        name="">
-        <color
-          rgba="0.3 0.3 0.3 1" />
-      </material>
-    </visual>
-    <collision>
-      <origin
-        xyz="0 0 0"
-        rpy="0 0 0" />
-      <geometry>
-        <mesh
-          filename="${mesh_path}canera_right_IR_ROS_frame.STL" />
-      </geometry>
-    </collision>
-  </link>
-  <joint
-    name="canera_right_IR_ROS_Joint"
-    type="fixed">
-    <origin
-      xyz="0.034005 -0.0475 0.014048"
+  </link>
+  <joint
+    name="camera_depth_joint"
+    type="fixed">
+    <origin
+      xyz="0 0 0"
       rpy="0 0 0" />
     <parent
       link="camera_link" />
     <child
-      link="canera_right_IR_ROS_frame" />
+      link="camera_depth_frame" />
+    <axis
+      xyz="0 0 0" />
+  </joint>
+  <joint
+    name="base_joint"
+    type="fixed">
+    <origin
+      xyz="-0.034005 -0.0475 -0.014048"
+      rpy="0 0 0" />
+    <parent
+      link="camera_link" />
+    <child
+      link="camera_botton_screw_frame" />
     <axis
       xyz="0 0 0" />
   </joint>
   <link
-    name="canera_left_IR_ROS_frame">
+    name="camera_right_ir_frame">
     <inertial>
       <origin
@@ -174,4 +151,57 @@
       <geometry>
         <mesh
+          filename="${mesh_path}canera_right_IR_ROS_frame.STL" />
+      </geometry>
+      <material
+        name="">
+        <color
+          rgba="0.3 0.3 0.3 1" />
+      </material>
+    </visual>
+    <collision>
+      <origin
+        xyz="0 0 0"
+        rpy="0 0 0" />
+      <geometry>
+        <mesh
+          filename="${mesh_path}canera_right_IR_ROS_frame.STL" />
+      </geometry>
+    </collision>
+  </link>
+  <joint
+    name="camera_right_ir_joint"
+    type="fixed">
+    <origin
+      xyz="0 -0.095 0"
+      rpy="0 0 0" />
+    <parent
+      link="camera_depth_frame" />
+    <child
+      link="camera_right_ir_frame" />
+    <axis
+      xyz="0 0 0" />
+  </joint>
+  <link
+    name="camera_left_ir_frame">
+    <inertial>
+      <origin
+        xyz="-0.0015782 9.8699E-08 -1.6899E-07"
+        rpy="0 0 0" />
+      <mass
+        value="0.00045313" />
+      <inertia
+        ixx="4.3406E-09"
+        ixy="-5.1012E-13"
+        ixz="-6.3511E-13"
+        iyy="4.8388E-09"
+        iyz="1.081E-12"
+        izz="4.8408E-09" />
+    </inertial>
+    <visual>
+      <origin
+        xyz="0 0 0"
+        rpy="0 0 0" />
+      <geometry>
+        <mesh
           filename="${mesh_path}canera_left_IR_ROS_frame.STL" />
       </geometry>
@@ -193,18 +223,18 @@
   </link>
   <joint
-    name="canera_left_IR_ROS_Joint"
-    type="fixed">
-    <origin
-      xyz="0.034005 0.0475 0.014048"
-      rpy="0 0 0" />
-    <parent
-      link="camera_link" />
-    <child
-      link="canera_left_IR_ROS_frame" />
+    name="camera_left_ir_joint"
+    type="fixed">
+    <origin
+      xyz="0 0 0"
+      rpy="0 0 0" />
+    <parent
+      link="camera_depth_frame" />
+    <child
+      link="camera_left_ir_frame" />
     <axis
       xyz="0 0 0" />
   </joint>
   <link
-    name="canera_RGB_ROS_frame">
+    name="camera_color_frame">
     <inertial>
       <origin
@@ -246,18 +276,18 @@
   </link>
   <joint
-    name="canera_RGB_ROS_Joint"
-    type="fixed">
-    <origin
-      xyz="0.034014 0.02375 0.014048"
-      rpy="0 0 0" />
-    <parent
-      link="camera_link" />
-    <child
-      link="canera_RGB_ROS_frame" />
+    name="camera_color_joint"
+    type="fixed">
+    <origin
+      xyz="9e-06 -0.02375 0"
+      rpy="0 0 0" />
+    <parent
+      link="camera_depth_frame" />
+    <child
+      link="camera_color_frame" />
     <axis
       xyz="0 0 0" />
   </joint>
   <link
-    name="canera_IMU_ROS_frame">
+    name="camera_imu_frame">
     <inertial>
       <origin
@@ -299,13 +329,13 @@
   </link>
   <joint
-    name="canera_IMU_ROS_Joint"
-    type="fixed">
-    <origin
-      xyz="0.019757 0.03619 0.013358"
-      rpy="0 0 0" />
-    <parent
-      link="camera_link" />
-    <child
-      link="canera_IMU_ROS_frame" />
+    name="camera_imu_joint"
+    type="fixed">
+    <origin
+      xyz="-0.014248 -0.01131 -0.00069"
+      rpy="0 0 0" />
+    <parent
+      link="camera_depth_frame" />
+    <child
+      link="camera_imu_frame" />
     <axis
       xyz="0 0 0" />

File: src/OrbbecSDK_ROS2/orbbec_description/urdf/gemini335Lg.urdf.xacro (robot description, xacro)
@@ -24,5 +24,5 @@
     <visual>
       <origin
-        xyz="0 0 0"
+        xyz="-0.0117149999999995 -0.0475 -0.0143111800025738"
         rpy="0 0 0" />
       <geometry>
@@ -87,8 +87,8 @@
   </link>
   <joint
-    name="camera_bottom_screw_frame"
-    type="fixed">
-    <origin
-      xyz="0 0 0"
+    name="camera_bottom_screw_joint"
+    type="fixed">
+    <origin
+      xyz="-0.0117149999999995 -0.0475 -0.0143111800025738"
       rpy="0 0 0" />
     <parent
@@ -100,5 +100,5 @@
   </joint>
   <link
-    name="camera_infra1_frame">
+    name="camera_left_ir_frame">
     <inertial>
       <origin
@@ -140,18 +140,18 @@
   </link>
   <joint
-    name="camera_infra1_frame"
-    type="fixed">
-    <origin
-      xyz="0.0117149999999995 0.0475 0.0143111800025738"
+    name="camera_left_ir_joint"
+    type="fixed">
+    <origin
+      xyz="0 0 0"
       rpy="0 0 0" />
     <parent
-      link="camera_bottom_screw_frame" />
-    <child
-      link="camera_infra1_frame" />
-    <axis
-      xyz="0 0 0" />
-  </joint>
-  <link
-    name="camera_infra1_optical_frame">
+      link="camera_depth_frame" />
+    <child
+      link="camera_left_ir_frame" />
+    <axis
+      xyz="0 0 0" />
+  </joint>
+  <link
+    name="camera_left_ir_optical_frame">
     <inertial>
       <origin
@@ -193,5 +193,5 @@
   </link>
   <joint
-    name="camera_infra1_optical_frame"
+    name="camera_left_ir_optical_joint"
     type="fixed">
     <origin
@@ -199,7 +199,7 @@
       rpy="-1.5707963267949 0 -1.5707963267949" />
     <parent
-      link="camera_infra1_frame" />
-    <child
-      link="camera_infra1_optical_frame" />
+      link="camera_left_ir_frame" />
+    <child
+      link="camera_left_ir_optical_frame" />
     <axis
       xyz="0 0 0" />
@@ -246,11 +246,11 @@
   </link>
   <joint
-    name="camera_color_frame"
-    type="fixed">
-    <origin
-      xyz="0.0117149999999995 0.02375 0.0143111800025738"
+    name="camera_color_joint"
+    type="fixed">
+    <origin
+      xyz="0 -0.023749999701976776 0"
       rpy="0 0 0" />
     <parent
-      link="camera_bottom_screw_frame" />
+      link="camera_depth_frame" />
     <child
       link="camera_color_frame" />
@@ -299,5 +299,5 @@
   </link>
   <joint
-    name="camera_color_optical_frame"
+    name="camera_color_optical_joint"
     type="fixed">
     <origin
@@ -312,5 +312,5 @@
   </joint>
   <link
-    name="camera_infra2_frame">
+    name="camera_right_ir_frame">
     <inertial>
       <origin
@@ -352,18 +352,18 @@
   </link>
   <joint
-    name="camera_infra2_frame"
-    type="fixed">
-    <origin
-      xyz="0.0117149999999995 -0.0475 0.0143111800025738"
+    name="camera_right_ir_joint"
+    type="fixed">
+    <origin
+      xyz="0 -0.095 0"
       rpy="0 0 0" />
     <parent
-      link="camera_bottom_screw_frame" />
-    <child
-      link="camera_infra2_frame" />
-    <axis
-      xyz="0 0 0" />
-  </joint>
-  <link
-    name="camera_infra2_optical_frame">
+      link="camera_depth_frame" />
+    <child
+      link="camera_right_ir_frame" />
+    <axis
+      xyz="0 0 0" />
+  </joint>
+  <link
+    name="camera_right_ir_optical_frame">
     <inertial>
       <origin
@@ -405,5 +405,5 @@
   </link>
   <joint
-    name="camera_infra2_optical_frame"
+    name="camera_right_ir_optical_joint"
     type="fixed">
     <origin
@@ -411,12 +411,12 @@
       rpy="-1.57079632679486 0 -1.5707963267949" />
     <parent
-      link="camera_infra2_frame" />
-    <child
-      link="camera_infra2_optical_frame" />
-    <axis
-      xyz="0 0 0" />
-  </joint>
-  <link
-    name="camera_IMU_frame">
+      link="camera_right_ir_frame" />
+    <child
+      link="camera_right_ir_optical_frame" />
+    <axis
+      xyz="0 0 0" />
+  </joint>
+  <link
+    name="camera_imu_frame">
     <inertial>
       <origin
@@ -458,13 +458,13 @@
   </link>
   <joint
-    name="camera_IMU_frame"
-    type="fixed">
-    <origin
-      xyz="-0.00253500000000046 0.036187989999999 0.0136240800025733"
+    name="camera_imu_joint"
+    type="fixed">
+    <origin
+      xyz="-0.01425 -0.011312 -0.0006871"
       rpy="0 0 0" />
     <parent
-      link="camera_bottom_screw_frame" />
-    <child
-      link="camera_IMU_frame" />
+      link="camera_depth_frame" />
+    <child
+      link="camera_imu_frame" />
     <axis
       xyz="0 0 0" />
@@ -511,11 +511,11 @@
   </link>
   <joint
-    name="camera_depth_frame"
-    type="fixed">
-    <origin
-      xyz="0.0117149999999995 0.0475 0.0143111800025738"
+    name="camera_depth_joint"
+    type="fixed">
+    <origin
+      xyz="0 0 0"
       rpy="0 0 0" />
     <parent
-      link="camera_bottom_screw_frame" />
+      link="camera_link" />
     <child
       link="camera_depth_frame" />

File: src/OrbbecSDK_ROS2/orbbec_description/urdf/gemini_335_336.urdf.xacro (robot description, xacro)
@@ -15,5 +15,5 @@
         </inertial>
         <visual>
-            <origin xyz="0 0 0" rpy="0 0 0" />
+            <origin xyz="-0.01587 -0.025 -0.0125" rpy="0 0 0" />
             <geometry>
                 <mesh filename="${mesh_path}camera_link.STL" />
@@ -55,5 +55,5 @@
     </link>
     <joint name="camera_bottom_screw_frame_joint" type="fixed">
-        <origin xyz="0 0 0" rpy="0 0 0" />
+        <origin xyz="-0.01587 -0.025 -0.0125" rpy="0 0 0" />
         <parent link="camera_link" />
         <child link="camera_bottom_screw_frame" />
@@ -86,6 +86,6 @@
     </link>
     <joint name="camera_left_ir_joint" type="fixed">
-        <origin xyz="0.01587 -0.025 0.0125" rpy="0 0 0" />
-        <parent link="camera_bottom_screw_frame" />
+        <origin xyz="0 0 0" rpy="0 0 0" />
+        <parent link="camera_depth_frame" />
         <child link="camera_left_ir_frame" />
         <axis xyz="0 0 0" />
@@ -116,6 +116,6 @@
     </link>
     <joint name="camera_left_ir_optical_joint" type="fixed">
-        <origin xyz="0.01587 -0.025 0.0125" rpy="-1.5707963267949 0 -1.5707963267949" />
-        <parent link="camera_bottom_screw_frame" />
+        <origin xyz="0 0 0" rpy="-1.5707963267949 0 -1.5707963267949" />
+        <parent link="camera_left_ir_frame" />
         <child link="camera_left_ir_optical_frame" />
         <axis xyz="0 0 0" />
@@ -147,6 +147,6 @@
     </link>
     <joint name="camera_right_ir_joint" type="fixed">
-        <origin xyz="0.01587 0.025 0.0125" rpy="0 0 0" />
-        <parent link="camera_bottom_screw_frame" />
+        <origin xyz="0 -0.05 0" rpy="0 0 0" />
+        <parent link="camera_depth_frame" />
         <child link="camera_right_ir_frame" />
         <axis xyz="0 0 0" />
@@ -177,6 +177,6 @@
     </link>
     <joint name="camera_right_ir_optical_joint" type="fixed">
-        <origin xyz="0.01587 0.025 0.0125" rpy="-1.5707963267949 0 -1.5707963267949" />
-        <parent link="camera_bottom_screw_frame" />
+        <origin xyz="0 0 0" rpy="-1.5707963267949 0 -1.5707963267949" />
+        <parent link="camera_right_ir_frame" />
         <child link="camera_right_ir_optical_frame" />
         <axis xyz="0 0 0" />
@@ -208,6 +208,6 @@
     </link>
     <joint name="camera_color_joint" type="fixed">
-        <origin xyz="0.017533 0.010995 0.012505" rpy="0 0 0" />
-        <parent link="camera_bottom_screw_frame" />
+        <origin xyz="0.001663 -0.014005 0.000005" rpy="0 0 0" />
+        <parent link="camera_depth_frame" />
         <child link="camera_color_frame" />
         <axis xyz="0 0 0" />
@@ -239,6 +239,6 @@
     </link>
     <joint name="camera_color_optical_joint" type="fixed">
-        <origin xyz="0.017533 0.010995 0.012505" rpy="-1.5707963267949 0 -1.5707963267949" />
-        <parent link="camera_bottom_screw_frame" />
+        <origin xyz="0 0 0" rpy="-1.5707963267949 0 -1.5707963267949" />
+        <parent link="camera_color_frame" />
         <child link="camera_color_optical_frame" />
         <axis xyz="0 0 0" />
@@ -270,6 +270,6 @@
     </link>
     <joint name="camera_depth_joint" type="fixed">
-        <origin xyz="0.01587 -0.025 0.0125" rpy="0 0 0" />
-        <parent link="camera_bottom_screw_frame" />
+        <origin xyz="0 0 0" rpy="0 0 0" />
+        <parent link="camera_link" />
         <child link="camera_depth_frame" />
         <axis xyz="0 0 0" />
@@ -299,6 +299,6 @@
     </link>
     <joint name="camera_depth_optical_joint" type="fixed">
-        <origin xyz="0.01587 -0.025 0.0125" rpy="-1.5707963267949 0 -1.5707963267949" />
-        <parent link="camera_bottom_screw_frame" />
+        <origin xyz="0 0 0" rpy="-1.5707963267949 0 -1.5707963267949" />
+        <parent link="camera_depth_frame" />
         <child link="camera_depth_optical_frame" />
         <axis xyz="0 0 0" />
